File: pcb-design/laser/prototype_adc2/prototype_adc2.kicad_pcb (KiCad board)
At the start: 4 copper layers, 37 x 26 mm, 59 parts, among them J1 Conn_01x01_Socket, J2 Conn_01x01_Socket, J3 Conn_01x01_Socket, J4 Conn_01x01_Socket, J5 Conn_01x01_Socket, J6 Conn_01x01_Socket, J7 Conn_01x01_Socket, J8 Conn_01x01_Socket, J9 Conn_01x01_Socket, U2 MCP1541T-I_TT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

Commit message: laser schematic AA cutoff fix
Other:
- board text added: "+9V"
- board text added: "-9V"
- board text added: "ADD 5V PIN FOR LEVEL SHIFTERS TO 3V3 MCUs"
- board text added: "FIX LASER FOOTPRINT"
- board text added: "TODO:"
- board text removed: "+5V"
- board text removed: "-5V"
Changed lines of the file:
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@@
     (effects (font (size 1 1) (thickness 0.2) bold) (justify left bottom mirror))
   )
-  (gr_text "+5V" (at 138.43 89.662 -270) (layer "B.SilkS")
+  (gr_text "+9V" (at 138.43 89.662 90) (layer "B.SilkS")
     (effects (font (size 1 1) (thickness 0.2) bold) (justify left bottom mirror))
   )
@@
     (effects (font (size 1 1) (thickness 0.2) bold) (justify left bottom mirror))
   )
-  (gr_text "-5V" (at 138.43 99.822 -270) (layer "B.SilkS")
+  (gr_text "-9V" (at 138.43 99.822 90) (layer "B.SilkS")
     (effects (font (size 1 1) (thickness 0.2) bold) (justify left bottom mirror))
   )
@@
     (effects (font (size 1 1) (thickness 0.2) bold) (justify left bottom))
   )
-  (gr_text "+5V" (at 137.16 89.662 270) (layer "F.SilkS")
+  (gr_text "+9V" (at 137.16 89.662 270) (layer "F.SilkS")
     (effects (font (size 1 1) (thickness 0.2) bold) (justify left bottom))
   )
@@
     (effects (font (size 1 1) (thickness 0.2) bold) (justify left bottom))
   )
-  (gr_text "-5V" (at 137.16 99.822 270) (layer "F.SilkS")
+  (gr_text "-9V" (at 137.16 99.822 270) (layer "F.SilkS")
     (effects (font (size 1 1) (thickness 0.2) bold) (justify left bottom))
   )
@@
     (effects (font (size 1 1) (thickness 0.2) bold) (justify left bottom))
   )
+  (gr_text "ADD 5V PIN FOR LEVEL SHIFTERS TO 3V3 MCUs" (at 174.006 99.412) (layer "Cmts.User")
+    (effects (font (size 1 1) (thickness 0.2) bold) (justify left bottom))
+  )
+  (gr_text "TODO:" (at 171.786 94.642) (layer "Cmts.User")
+    (effects (font (size 1 1) (thickness 0.2) bold) (justify left bottom))
+  )
+  (gr_text "FIX LASER FOOTPRINT" (at 174.006 97.052) (layer "Cmts.User")
+    (effects (font (size 1 1) (thickness 0.2) bold) (justify left bottom))
+  )

Commit message: fixed laser footprint on pcb
Parts:
- D1: moved to B.Cu
Routing:
- net /ld_i: track 6.42 -> 8.01 mm
- net /pd_out: track 15.1 -> 15.9 mm
Other:
- board text removed: "FIX LASER FOOTPRINT"
